File: Electronics/Network Weather Board.sch (KiCad schematic (older format))
At the start: 7 parts

Commit message: Added in the W5100 Ehternet chip and fixed some issues with net-lists
Parts:
- added C? (x2): 18pF, symbol C
- added GREEN (x2), RED, YELLOW: LED, symbol LED
- added JP? (x2): JUMPER, symbol JUMPER
- added R1, R2, R3, R4: 1k, symbol R
- added R17: 10k, symbol R
- added R?: 12k, symbol R
- added R?: 300, symbol R
- added R?: 1M, symbol R
- added U?: W5100, symbol W5100
- added X?: 25MHz, symbol CRYSTAL
Connections:
- net labels added: *CS, +3.3V, 1V8, 1V8A, 3V3A, FDX LED, INT, IO2, LINK LED, RESET, RXIN, RXIP, SCLK, TXON, TXOP
- wire segments 25 -> 107
- no-connect marks 0 -> 33
Other:
- note added: "ARDUINO (ATMEGA 328P)"
- note added: "ETHERNET (W5100)"
- moved on the sheet: C1, C2, C3, IC?, R1, RESET, X?

Commit message: The schematic should be done now =)
Parts:
- added C1, C11: 10uF, symbol C
- added C10, C12, C13, C14, C17, C2, C3, C4, C5, C8: 0.1uF, symbol C
- added J1: RJ45-MAG, symbol RJ45-MAG
- added L1, L2, L3: 1uH, symbol INDUCTOR
- added R2, R3, R5, R6: 49.9, symbol R
- added R4, R7: 330, symbol R
- added R8, R9: 4.7k, symbol R
- gave numbers to parts that had none: 11
- renumbered C1 to C6, C2 to C7, C3 to C9, GREEN to GREEN1, GREEN to GREEN2, R17 to R13, R1 to R14, R2 to R15, R3 to R16, R4 to R17, RED to RED1, RESET to RESET1, YELLOW to YELLOW1
Connections:
- net labels added: AD0, AD1, AD2, AD3, AD4, AD5, AD6, AD7, DTR, IO0, IO1, IO3, IO4, IO5, IO6, IO7, IO8, IO9, SCL, SDA
- net labels removed: CLK, SCK
- wire segments 107 -> 193
- no-connect marks 33 -> 35
Other:
- note added: "DECOUPLING"
- note added: "MAGJACK"
- moved on the sheet: C6, C7, C9, IC1, R1, RESET1, X1
